Commit message: Add ros2_control differential drive configuration

File: ros2_ws/src/shelf_description/urdf/ros2_control.xacro (robot description, xacro)
@@ -1,4 +1,20 @@
 <?xml version="1.0"?>
 <robot xmlns:xacro="http://www.ros.org/wiki/xacro">
-  <!-- ros2_control will be added in Phase 2. -->
+  <xacro:macro name="shelf_robot_ros2_control">
+    <ros2_control name="ShelfRobotSystem" type="system">
+      <hardware>
+        <plugin>mock_components/GenericSystem</plugin>
+      </hardware>
+      <joint name="left_wheel_joint">
+        <command_interface name="velocity"/>
+        <state_interface name="position"/>
+        <state_interface name="velocity"/>
+      </joint>
+      <joint name="right_wheel_joint">
+        <command_interface name="velocity"/>
+        <state_interface name="position"/>
+        <state_interface name="velocity"/>
+      </joint>
+    </ros2_control>
+  </xacro:macro>
 </robot>

File: ros2_ws/src/shelf_description/urdf/shelf_robot.urdf.xacro (robot description, xacro)
@@ -8,3 +8,4 @@
   <xacro:include filename="ros2_control.xacro"/>
   <xacro:include filename="gazebo.xacro"/>
+  <xacro:shelf_robot_ros2_control/>
 </robot>
